Commit message: chore: add bug

File: roverto_description/urdf/roverto.urdf.xacro (robot description, xacro)
@@ -1,4 +1,5 @@
 <?xml version="1.0"?>
 <robot name="roverto" xmlns:xacro="http://www.ros.org/wiki/xacro">
+  <!-- ================= CONSTANTS & DIMENSIONS ================= -->
   <!-- Chassis -->
   <xacro:property name="chassis_length" value="0.20"/>
@@ -14,5 +15,9 @@
   <xacro:property name="wheel_y_offset" value="0.1135"/>
   <xacro:property name="ground_clearance" value="0.015"/>
-  <!-- Inertia Macros -->
+  <!-- LD19 LiDAR -->
+  <xacro:property name="lidar_radius" value="0.019"/>
+  <xacro:property name="lidar_height" value="0.0335"/>
+  <xacro:property name="lidar_mass"   value="0.042"/>
+  <!-- ================= INERTIA MACROS ================= -->
   <xacro:macro name="box_inertia" params="m x y z">
     <inertial>
@@ -31,5 +36,5 @@
     </inertial>
   </xacro:macro>
-  <!-- Links -->
+  <!-- ================= BASE FOOTPRINT & BASE LINK ================= -->
   <link name="base_footprint"/>
   <joint name="base_joint" type="fixed">
@@ -89,3 +94,57 @@
   <xacro:wheel prefix="rear_left"   x_reflect="-1" y_reflect="1" />
   <xacro:wheel prefix="rear_right"  x_reflect="-1" y_reflect="-1" />
+  <!-- ================= LIDAR (LD19) LINK & JOINT ================= -->
+  <joint name="lidar_joint" type="fixed">
+    <parent link="base_link"/>
+    <child link="laser_frame"/>
+    <origin xyz="0.0 0.0 ${chassis_height + (lidar_height / 2.0)}" rpy="0 0 0"/>
+  </joint>
+  <link name="laser_frame">
+    <visual>
+      <origin xyz="0 0 0" rpy="0 0 0"/>
+      <geometry>
+        <cylinder radius="${lidar_radius}" length="${lidar_height}"/>
+      </geometry>
+      <material name="lidar_blue">
+        <color rgba="0.1 0.4 0.8 1.0"/>
+      </material>
+    </visual>
+    <collision>
+      <origin xyz="0 0 0" rpy="0 0 0"/>
+      <geometry>
+        <cylinder radius="${lidar_radius}" length="${lidar_height}"/>
+      </geometry>
+    </collision>
+    <xacro:cylinder_inertia m="${lidar_mass}" r="${lidar_radius}" h="${lidar_height}"/>
+  </link>
+  <!-- ================= GAZEBO SENSOR PLUGIN ================= -->
+  <gazebo reference="laser_frame">
+    <sensor name="lidar" type="gpu_lidar">
+      <always_on>true</always_on>
+      <visualize>true</visualize>
+      <update_rate>10</update_rate>
+      <topic>scan</topic>
+      <gz_frame_id>laser_frame</gz_frame_id>
+      <lidar>
+        <scan>
+          <horizontal>
+            <samples>450</samples>
+            <resolution>1</resolution>
+            <min_angle>-3.14159265</min_angle>
+            <max_angle>3.14159265</max_angle>
+          </horizontal>
+        </scan>
+        <range>
+          <min>0.02</min>
+          <max>12.0</max>
+          <resolution>0.01</resolution>
+        </range>
+        <noise>
+          <type>gaussian</type>
+          <mean>0.0</mean>
+          <stddev>0.01</stddev>
+        </noise>
+      </lidar>
+    </sensor>
+  </gazebo>
 </robot>

Commit message: chore: add differential drive

File: roverto_description/urdf/roverto.urdf.xacro (robot description, xacro)
@@ -15,4 +15,12 @@
   <xacro:property name="wheel_y_offset" value="0.1135"/>
   <xacro:property name="ground_clearance" value="0.015"/>
+  <!-- Skid-steer calibration -->
+  <!-- Wheel friction used in simulation (isotropic). Lower = easier to turn in place. -->
+  <xacro:property name="wheel_mu" value="0.4"/>
+  <!-- Effective track width = geometric track * slip_factor.
+       Start at 1.0, then do a 360 deg in-place rotation test and set:
+       slip_factor = commanded_yaw / actual_yaw  (typically 1.2 - 1.8 for skid-steer) -->
+  <xacro:property name="slip_factor" value="1.0"/>
+  <xacro:property name="wheel_separation" value="${2.0 * wheel_y_offset * slip_factor}"/>
   <!-- LD19 LiDAR -->
   <xacro:property name="lidar_radius" value="0.019"/>
@@ -20,6 +28,8 @@
   <xacro:property name="lidar_mass"   value="0.042"/>
   <!-- ================= INERTIA MACROS ================= -->
+  <!-- Box inertia, with the center of mass at the box center (box origin sits at z/2 in base_link) -->
   <xacro:macro name="box_inertia" params="m x y z">
     <inertial>
+      <origin xyz="0 0 ${z / 2.0}" rpy="0 0 0"/>
       <mass value="${m}"/>
       <inertia ixx="${(m/12.0) * (y*y + z*z)}" ixy="0.0" ixz="0.0"
@@ -28,4 +38,5 @@
     </inertial>
   </xacro:macro>
+  <!-- Cylinder with its axis along Z (used by the LiDAR) -->
   <xacro:macro name="cylinder_inertia" params="m r h">
     <inertial>
@@ -34,4 +45,13 @@
                iyy="${(m/12.0) * (3*r*r + h*h)}" iyz="0.0"
                izz="${(m/2.0) * (r*r)}"/>
+    </inertial>
+  </xacro:macro>
+  <!-- Wheel inertia: spin axis is Y (matches joint axis 0 1 0 and the visual/collision rotation) -->
+  <xacro:macro name="wheel_inertia" params="m r h">
+    <inertial>
+      <mass value="${m}"/>
+      <inertia ixx="${(m/12.0) * (3*r*r + h*h)}" ixy="0.0" ixz="0.0"
+               iyy="${(m/2.0) * (r*r)}" iyz="0.0"
+               izz="${(m/12.0) * (3*r*r + h*h)}"/>
     </inertial>
   </xacro:macro>
@@ -80,5 +100,5 @@
         </geometry>
       </collision>
-      <xacro:cylinder_inertia m="${wheel_mass}" r="${wheel_radius}" h="${wheel_width}"/>
+      <xacro:wheel_inertia m="${wheel_mass}" r="${wheel_radius}" h="${wheel_width}"/>
     </link>
     <joint name="${prefix}_wheel_joint" type="continuous">
@@ -88,4 +108,9 @@
       <axis xyz="0 1 0"/>
     </joint>
+    <!-- Wheel/ground friction (needed for skid-steer to be able to turn in simulation) -->
+    <gazebo reference="${prefix}_wheel_link">
+      <mu1>${wheel_mu}</mu1>
+      <mu2>${wheel_mu}</mu2>
+    </gazebo>
   </xacro:macro>
   <!-- Instantiate 4 Wheels -->
@@ -94,5 +119,5 @@
   <xacro:wheel prefix="rear_left"   x_reflect="-1" y_reflect="1" />
   <xacro:wheel prefix="rear_right"  x_reflect="-1" y_reflect="-1" />
-  <!-- ================= LIDAR (LD19) LINK & JOINT ================= -->
+  <!--  LIDAR (LD19) LINK & JOINT  -->
   <joint name="lidar_joint" type="fixed">
     <parent link="base_link"/>
@@ -118,5 +143,5 @@
     <xacro:cylinder_inertia m="${lidar_mass}" r="${lidar_radius}" h="${lidar_height}"/>
   </link>
-  <!-- ================= GAZEBO SENSOR PLUGIN ================= -->
+  <!--  GAZEBO SENSOR PLUGIN  -->
   <gazebo reference="laser_frame">
     <sensor name="lidar" type="gpu_lidar">
@@ -148,3 +173,40 @@
     </sensor>
   </gazebo>
+  <!--  GAZEBO DIFFERENTIAL DRIVE PLUGIN -->
+  <gazebo>
+    <plugin
+      filename="gz-sim-diff-drive-system"
+      name="gz::sim::systems::DiffDrive">
+      <!-- Left and Right wheel joints (skid-steer 4-wheel configuration) -->
+      <left_joint>front_left_wheel_joint</left_joint>
+      <left_joint>rear_left_wheel_joint</left_joint>
+      <right_joint>front_right_wheel_joint</right_joint>
+      <right_joint>rear_right_wheel_joint</right_joint>
+      <!-- Kinematics geometric track (2 * wheel_y_offset = 0.227) scaled by slip_factor -->
+      <wheel_separation>${wheel_separation}</wheel_separation>
+      <wheel_radius>${wheel_radius}</wheel_radius>
+      <!-- Limits -->
+      <max_linear_acceleration>1.0</max_linear_acceleration>
+      <max_angular_acceleration>2.0</max_angular_acceleration>
+      <min_linear_velocity>-0.5</min_linear_velocity>
+      <max_linear_velocity>0.5</max_linear_velocity>
+      <min_angular_velocity>-1.5</min_angular_velocity>
+      <max_angular_velocity>1.5</max_angular_velocity>
+      <!-- Topics & Frames -->
+      <topic>/cmd_vel</topic>
+      <odom_topic>/odom</odom_topic>
+      <frame_id>odom</frame_id>
+      <child_frame_id>base_footprint</child_frame_id>
+      <odom_publisher_frequency>30</odom_publisher_frequency>
+      <tf_topic>/tf</tf_topic>
+    </plugin>
+  </gazebo>
+  <!--  GAZEBO JOINT STATE PUBLISHER (wheel joint angles for robot_state_publisher / RViz) -->
+  <gazebo>
+    <plugin
+      filename="gz-sim-joint-state-publisher-system"
+      name="gz::sim::systems::JointStatePublisher">
+      <topic>joint_states</topic>
+    </plugin>
+  </gazebo>
 </robot>
